Commit message: working for LAFAN

File: holosoma-main/src/holosoma_retargeting/holosoma_retargeting/models/ch_robot/ch_robot_10dof.urdf (robot description, URDF)
Before this commit: robot ch_robot, 20 links, 19 joints
Links:
- added link left_ankle_marker, mass 0.001; visual sphere radius=0.01
- added link right_ankle_marker, mass 0.001; visual sphere radius=0.01
Joints:
- added joint left_ankle_marker_joint: type fixed, parent left_foot, child left_ankle_marker, origin xyz=0 0 0 rpy=0 0 0
- added joint right_ankle_marker_joint: type fixed, parent right_foot, child right_ankle_marker, origin xyz=0 0 0 rpy=0 0 0
